Commit message: update arm constraints

File: urdf/braccio_arm.urdf (robot description, URDF)
Before this commit: robot visual, 8 links, 7 joints
Joints:
- joint gripper_joint: limit lower=1.217 upper=1.5708 effort=1000.0 velocity=1.0 -> lower=0.18 upper=1.27 effort=1000.0 velocity=1.0

Commit message: get gripper working;

File: urdf/braccio_arm.urdf (robot description, URDF)
Before this commit: robot visual, 8 links, 7 joints
Joints:
- joint sub_gripper_joint: limit lower=1.5708 upper=2.7876 effort=1000.0 velocity=1.0 -> lower=0.18 upper=1.27 effort=1000.0 velocity=1.0
- joint wrist_roll_joint: origin xyz=0 0.0 0.06 rpy=0 0 0 -> xyz=0 0.0 0.06 rpy=0 0 1.5708
